File: kicad/lcd_large/lcd2wire.kicad_pcb (KiCad board)
At the start: 2 copper layers, 68.2 x 25.7 mm, 16 parts, among them J1 LCD2Wire, J2 615004141121, J3 Conn_01x16, U1 AZ1117-5.0, U2 74LS174

Commit message: Update text on lcd2wire large board
Other:
- board text added: "SB.ATVIE.0921"
- board text removed: "www.realtimesolutions.at"
